File: nova_v2/schematics/electronics/nova_v2.kicad_sch (KiCad schematic)
At the start: 15 parts, among them M2 Motor_DC, Q1 BC547, SW1 SW_Push, SW2 SW_SPDT, U1 TP4056-42-ESOP8, U2 XIAO-ESP32-S3-SMD

Commit message: fixing the electronics schematics
Parts:
- removed D3: D, Seeed Studio XIAO SAMD21 (Pre-Soldered)_v2.1:C0402, symbol Device:D
- removed U1: TP4056-42-ESOP8, Package_SO:SOIC-8-1EP_3.9x4.9mm_P1.27mm_EP2.41x3.3mm_ThermalVias, symbol Battery_Management:TP4056-42-ESOP8
- added R3, R5: 220k, symbol Device:R
- C1: value 100nF -> 104nF
Connections:
- net 3V3: now also U2.10 (D9); no longer U2.4 (D3)
- net GND: now also SW1.1, R5.1; no longer SW1.2
- net HAPTIC: now also U2.2 (D1); no longer U2.5 (D4)
- net SCK: now also U2.9 (D8); no longer U2.3 (D2)
- net V_in: now also R3.1
- net WS: now also U2.11 (D10); no longer U2.2 (D1)
- net at U2.1 (D0): now also R3.2, R5.2
- net at R2.2: now also U2.4 (D3); no longer U2.8 (D7)
- net at R1.2: now also U2.5 (D4); no longer U2.9 (D8)
- new net: SW1.2, U2.3 (D2)
- no-connect marks 14 -> 13
Other:
- note removed: "Just in case - battery charger module"
- company: (none) -> Project Nova
- title: (none) -> Nova Version 2 Electronics Schematic
- moved on the sheet: D1, D2, R1, R2, SW1, U2
